File: simple_drone_kicad/simple_drone.kicad_sch (KiCad schematic)
At the start: 35 parts, among them P1 USB_C_Plug_USB2.0, Q1 FDN340P, U1 BMI088, U2 BMP581, U3 FT260S-U, U4 LMV358, Y1 Crystal_GND23

Commit message: finished initial schematic
Need to review, finish minor things,
fix TODOs
🤓🤓🤓
Parts:
- removed C? (x2): 0.1uF, symbol Device:C
- removed U1: BMI088, QFN_BMI085_BOS, symbol 2024-07-02_03-58-38:BMI088
- added D2, D3: LED, symbol Device:LED
- added IC1: ICM-20948, QFN40P300X300X105-25N-D, symbol ICM-20948:ICM-20948
- added J1, J2, J3, J4, J9: Conn_01x02, symbol Connector_Generic:Conn_01x02
- added J5, J6: Conn_01x04, symbol Connector_Generic:Conn_01x04
- added J7: Conn_01x06, symbol Connector_Generic:Conn_01x06
- added J8: Conn_01x03, symbol Connector_Generic:Conn_01x03
- added PWM1: PCA9685BS, Package_DFN_QFN:QFN-28-1EP_6x6mm_P0.65mm_EP4.25x4.25mm, symbol Driver_LED:PCA9685BS
- added R3, R4: 10k, symbol Device:R
- added R5, R6: 330, symbol Device:R
- added R7, R8: 5.1k, symbol Device:R
- added U5: M24C01-FMN, Package_SO:SOIC-8_3.9x4.9mm_P1.27mm, symbol Memory_EEPROM:M24C01-FMN
- R1: value R -> 330
- R2: value R -> 5.1k
- gave numbers to parts that had none: 21
Connections:
- net +12V: now also R3.1
- net +3.3V: now also U3.10 (VCCIO), U3.26 (VOUT3V3), U3.5 (DEBUGGER), U3.6 (STEST_RSTN), D2.2 (A), D3.2 (A), J5.1 (Pin_1), PWM1.25 (VDD), U5.8 (VCC)
- net +5V: now also C8.2, L1.2, U6.4 (FB), J7.1 (Pin_1), J9.1 (Pin_1)
- net GND: now also U3.23 (GND), U3.28 (AGND), U3.8 (DCNF0), U3.9 (DCNF1), IC1.18 (GND), J1.2 (Pin_2), J2.2 (Pin_2), J3.2 (Pin_2), J4.2 (Pin_2), J5.4 (Pin_4), J6.4 (Pin_4), J7.6 (Pin_6), J8.3 (Pin_3), J9.2 (Pin_2), PWM1.1 (A3), PWM1.11 (VSS), PWM1.2 (A4), PWM1.20 (~{OE}), PWM1.21 (A5), PWM1.26 (A0), PWM1.27 (A1), PWM1.28 (A2), PWM1.29 (VSS), R4.2, R7.2, U5.1 (E0), U5.2 (E1), U5.3 (E2), U5.4 (VSS)
- net SPI1_MISO: now also J6.1 (Pin_1)
- net SPI1_MOSI: now also J6.2 (Pin_2)
- net SPI1_SCK: now also J6.3 (Pin_3)
- net SPI2_SCK: now also U7.52 (PB13); no longer U7.47 (PB10)
- net USBVCC: now also R8.1
- net BAR_INT: now reaches U2.7 (INT)
- net USART2_TX: now reaches U7.25 (PA2)
- net USART2_TX: now also J7.3 (Pin_3)
- net USART2_RX: now reaches U7.26 (PA3)
- net USART2_RX: now also J7.2 (Pin_2)
- net USART3_RX: now reaches U7.48 (PB11)
- net USART3_RX: now also J8.1 (Pin_1)
- net I2C3_SDA: now reaches U7.66 (PC9)
- net I2C3_SDA: now also PWM1.24 (SDA)
- net I2C3_SCL: now reaches U7.67 (PA8)
- net I2C3_SCL: now also PWM1.23 (SCL)
- net SWDIO: now reaches U7.72 (PA13)
- net SWDIO: now also J5.2 (Pin_2)
- net SWDCLK: now reaches U7.76 (PA14)
- net SWDCLK: now also J5.3 (Pin_3)
- net SPI3_MOSI: now reaches U7.78 (PC10)
- net SPI3_MOSI: now also IC1.24 (SDA_/_SDI)
- net SPI3_MISO: now reaches U7.79 (PC11)
- net SPI3_MISO: now also IC1.9 (SDO_/_AD0)
- net SPI3_SCK: now reaches U7.80 (PC12)
- net I2C1_WC: now reaches U7.91 (PB5)
- net I2C1_WC: now also U5.7 (~{WC})
- net I2C1_SCL: now reaches U7.92 (PB6)
- net I2C1_SCL: now also U5.6 (SCL)
- net I2C1_SDA: now reaches U7.93 (PB7)
- net I2C1_SDA: now also U5.5 (SDA)
- net at P1.B5 (VCONN): now also R7.1
- net TX_LED: now reaches U3.11 (DIO0)
- net TX_LED: now also R5.2
- net at U3.2 (VBUS_DET): now also R8.2
- net RX_LED: now reaches U3.3 (DIO12)
- net RX_LED: now also R6.2
- net reset: now reaches U3.7 (RESETN)
- net SPI1_CSB1: no longer names the net of U7.29 (PA4)
- net SPI1_CSB2: no longer names the net of U7.33 (PC4)
- new net: D2.1 (K), R5.1
- new net: R3.2, R4.1, U4.3 (+)
- new net: D3.1 (K), R6.1
- new net IMU_INT: IC1.12 (INT1)
- new net PWM_1: J1.1 (Pin_1), PWM1.3 (LED0)
- new net PWM_2: J2.1 (Pin_1), PWM1.4 (LED1)
- new net PWM_3: J3.1 (Pin_1), PWM1.5 (LED2)
- new net PWM_4: J4.1 (Pin_1), PWM1.6 (LED3)
- new net USART3_TX: J8.2 (Pin_2), U7.47 (PB10)
- no-connect marks 3 -> 39
Other:
- note added: "9-axis IMU"
- note added: "EEPROM"
- note added: "ESC"
- note added: "ESC connections (dupont 2x1)"
- note added: "GNSS HolyBro 6 pin jst gh"
- note added: "Jetson nano 4x1 jst gh"
- note added: "LEDs"
- note added: "TODO: add i2c pullup resistors TODO: fix ERC TODO: assign footprints to symbols TODO: review schematic, need 2nd eye"
- note added: "TODO: add reverse polarity protection"
- note added: "debug 4x1 dupont"
- note added: "flysky fs-ia6b (iBus mode)"
- note removed: "IMU"
- note removed: "hookup imu intr pins to mcu (TODO)"
- moved on the sheet: C1, C10, C11, C12, C13, C14, C15, C16, C17, C2, C3, C4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

Commit message: fix erc errors, i2c pullup
Parts:
- added C18, C19: 2.2uF, Capacitor_SMD:C_0805_2012Metric, symbol Device:C
- added C20, C21: 0.1uF, symbol Device:C
- added R10: 10k, symbol Device:R
- added R9: 15k, symbol Device:R
- R3: value 10k -> 15k
Connections:
- net +3.3V: now also IC1.13 (VDD), U7.21 (VREF+), C20.2, R9.1
- net BAR_INT: now also U7.97 (PE0)
- net GND: now also IC1.20 (RESV_2), C18.2, C19.2, C20.1, C21.2, R10.2
- net IMU_INT: now also U7.98 (PE1)
- net SPI3_SCK: now also IC1.23 (SCL_/_SCLK)
- net VCAP_1: now reaches U7.49 (VCAP_1)
- net VCAP_1: now also C19.1
- net VCAP_2: now reaches U7.73 (VCAP_2)
- net VCAP_2: now also C18.1
- net at IC1.10 (REGOUT): now also C21.1
- net at IC1.8 (VDDIO): now also R10.1, R9.2
- no-connect marks 39 -> 100
Other:
- moved on the sheet: U4A
